Commit message: [WIP] fix examples

File: src/curobo/content/assets/robot/xarm_description/urdf/xarm7.urdf (robot description, URDF)
Before this commit: robot xarm7, 15 links, 14 joints
Joints:
- added joint left_finger_fixed_joint: type fixed, parent left_finger, child left_inner_knuckle, origin xyz=0 0.0205 0.027 rpy=0 0 0
- added joint right_finger_fixed_joint: type fixed, parent right_finger, child right_inner_knuckle, origin xyz=0 -0.0205 0.027 rpy=0 0 0

Commit message: fix

File: src/curobo/content/assets/robot/xarm_description/urdf/xarm7.urdf (robot description, URDF)
Before this commit: robot xarm7, 15 links, 16 joints
Links:
- added link fingertip_centered, mass 0.0001
Joints:
- added joint fingertip_fixed_joint: type None, parent xarm_gripper_base_link, child fingertip_centered, origin xyz=0 0 0.1455 rpy=0 0 0
